Commit message: fix parameters - rviz showing images

File: urdf/udacity_bot.xacro (robot description, xacro)
@@ -176,5 +176,5 @@
   </link>
   <joint type="fixed" name="camera_joint">
-    <origin xyz="0.2 0 0" rpy="0 0 0"/>
+    <origin xyz="0.2 0 0.1" rpy="0 0 0"/>
     <child link="camera"/>
     <parent link="chassis"/>

Commit message: got more loop closures

File: urdf/udacity_bot.xacro (robot description, xacro)
@@ -176,5 +176,5 @@
   </link>
   <joint type="fixed" name="camera_joint">
-    <origin xyz="0.2 0 0.1" rpy="0 0 0"/>
+    <origin xyz="0.2 0 0.05" rpy="0 0 0"/>
     <child link="camera"/>
     <parent link="chassis"/>

Commit message: fix camera and laser positions

File: urdf/udacity_bot.xacro (robot description, xacro)
@@ -176,5 +176,5 @@
   </link>
   <joint type="fixed" name="camera_joint">
-    <origin xyz="0.2 0 0.05" rpy="0 0 0"/>
+    <origin xyz="0.225 0 0.005" rpy="0 0 0"/>
     <child link="camera"/>
     <parent link="chassis"/>
@@ -207,5 +207,5 @@
   </link>
   <joint type="fixed" name="hokuyo_joint">
-    <origin xyz="0.15 0 0.1" rpy="0 0 0"/>
+    <origin xyz="0.1 0 0.08" rpy="0 0 0"/>
     <child link="hokuyo"/>
     <parent link="chassis"/>

Commit message: add kinect.dae & camera rgbd transform

File: urdf/udacity_bot.xacro (robot description, xacro)
@@ -160,13 +160,13 @@
     </inertial>
     <collision name='collision'>
-      <origin xyz="0 0 0" rpy=" 0 0 0"/>
-      <geometry>
-        <box size="0.05 0.05 0.05"/>
-      </geometry>
-    </collision>
-    <visual>
       <origin xyz="0 0 0" rpy="0 0 0"/>
       <geometry>
-        <box size=".05 0.05 0.05"/>
+        <box size="0.073 0.276 0.072"/>
+      </geometry>
+    </collision>
+    <visual>
+      <origin xyz="0 0 0" rpy="0 0 0"/>
+      <geometry>
+	<mesh filename="package://slam_project/meshes/kinect.dae" />
       </geometry>
       <material name="red">
@@ -179,4 +179,10 @@
     <child link="camera"/>
     <parent link="chassis"/>
+  </joint>
+  <link name="camera_rgbd_frame" />
+  <joint type="fixed" name="camera_rgbd_joint">
+    <origin xyz="0 0 0" rpy="-1.5707 0 -1.5707"/>
+    <parent link="camera"/>
+    <child link="camera_rgbd_frame"/>
   </joint>
   <link name='hokuyo'>

Commit message: fix camera_rgbd_frame

File: urdf/udacity_bot.xacro (robot description, xacro)
@@ -162,5 +162,5 @@
       <origin xyz="0 0 0" rpy="0 0 0"/>
       <geometry>
-        <box size="0.073 0.276 0.072"/>
+	<sphere radius="0.05" />
       </geometry>
     </collision>
@@ -168,5 +168,6 @@
       <origin xyz="0 0 0" rpy="0 0 0"/>
       <geometry>
-	<mesh filename="package://slam_project/meshes/kinect.dae" />
+	<!--<mesh filename="package://slam_project/meshes/kinect.dae" /> -->
+	<sphere radius="0.05" />
       </geometry>
       <material name="red">
@@ -198,5 +199,5 @@
       <origin xyz="0 0 0" rpy=" 0 0 0"/>
       <geometry>
-        <box size="0.1 0.1 0.1"/>
+        <sphere radius="0.05"/>
       </geometry>
     </collision>
@@ -204,6 +205,6 @@
       <origin xyz="0 0 0" rpy="0 0 0"/>
       <geometry>
-        <mesh filename="package://slam_project/meshes/hokuyo.dae"/>
-        <!-- <box size=".1"/> -->
+        <!--<mesh filename="package://slam_project/meshes/hokuyo.dae"/>-->
+        <sphere radius=".05"/>
       </geometry>
       <material name="blue">
